Commit message: Added inertia tags

File: description/urdf/urdf.xacro (robot description, xacro)
@@ -23,4 +23,7 @@
       </geometry>
     </collision>
+    <xacro:inertial_cylinder mass="0.5" length="${1.7  * 0.001}" radius="${50 * 0.001}">
+      <origin xyz="0 0 0" rpy="0 0 0"/>
+    </xacro:inertial_cylinder>
 </link>
 <joint name="chassis_joint" type="fixed">
@@ -58,4 +61,7 @@
     </geometry>
   </collision>
+  <xacro:inertial_cylinder mass="0.2" length="${10  * 0.001}" radius="${21 * 0.001}">
+    <origin xyz="0 ${-5 * 0.001} ${5 * 0.001}" rpy="${pi/2} 0 0"/>
+  </xacro:inertial_cylinder>
 </link>
 <joint name="left_wheel_joint" type="continuous">
@@ -136,4 +142,13 @@
     <material name="yellow"/>
   </visual>
+  <collision>
+    <origin xyz="0 ${-5 * 0.001} ${5 * 0.001}" rpy="${pi/2} 0 0"/>
+    <geometry>
+      <cylinder length="${10 * 0.001}" radius="${21 * 0.001}"/>
+    </geometry>
+  </collision>
+  <xacro:inertial_cylinder mass="0.2" length="${10  * 0.001}" radius="${21 * 0.001}">
+    <origin xyz="0 ${-5 * 0.001} ${5 * 0.001}" rpy="${pi/2} 0 0"/>
+  </xacro:inertial_cylinder>
 </link>
 <joint name="right_wheel_joint" type="continuous">
@@ -211,4 +226,7 @@
     </geometry>
   </collision>
+  <xacro:inertial_cylinder mass="0.2" length="${10  * 0.001}" radius="${21 * 0.001}">
+    <origin xyz="${42 * 0.001} ${12 * 0.001} ${-11.7 * 0.001}" rpy="0 0 0"/>
+  </xacro:inertial_cylinder>
 </link>
 <joint name="caster_wheel_joint" type="fixed">

Commit message: I'm back

File: description/urdf/urdf.xacro (robot description, xacro)
@@ -5,4 +5,5 @@
 <xacro:include filename="$(find cobalt)/description/urdf/urdf.trans" />
 <xacro:include filename="$(find cobalt)/description/urdf/urdf.gazebo" />
+<xacro:include filename="$(find cobalt)/description/urdf/control.xacro" />
 <!-- Base link -->
 <link name="base_link">
@@ -11,5 +12,5 @@
 <link name="chassis">
     <visual>
-        <origin xyz="0 0 0" rpy="0 0 0"/>
+        <origin xyz="0 0 ${1.7 * 0.001}" rpy="${pi} 0 0"/>
         <geometry>
           <mesh filename="file://$(find cobalt)/description/meshes/base_link.stl" scale="0.001 0.001 0.001"/>
@@ -20,8 +21,8 @@
       <origin xyz="0 0 0" rpy="0 0 0"/>
       <geometry>
-        <cylinder length="${1.7 * 0.001}" radius="${50 * 0.001}"/>
+        <cylinder length="${26 * 0.001}" radius="${50 * 0.001}"/>
       </geometry>
     </collision>
-    <xacro:inertial_cylinder mass="0.5" length="${1.7  * 0.001}" radius="${50 * 0.001}">
+    <xacro:inertial_cylinder mass="0.068" length="${1.7  * 0.001}" radius="${50 * 0.001}">
       <origin xyz="0 0 0" rpy="0 0 0"/>
     </xacro:inertial_cylinder>
@@ -30,24 +31,33 @@
     <parent link="base_link"/>
     <child link="chassis"/>
-    <origin xyz="0 0 0"/>
+    <origin xyz="0 0 ${-6.6 * 0.001}"/>
+</joint>
+<link name="battery">
+    <visual>
+        <origin xyz="0 0 0" rpy="0 0 0"/>
+        <geometry>
+            <mesh filename="file://$(find cobalt)/description/meshes/battery.stl" scale="0.001 0.001 0.001"/>
+        </geometry>
+        <material name="black"/>
+    </visual>
+    <collision>
+      <origin xyz="0 0 0" rpy="0 0 0"/>
+      <geometry>
+        <box size="${28 * 0.001} ${60 * 0.001} ${20 * 0.001}"/>
+      </geometry>
+    </collision>
+    <xacro:inertial_box mass="0.063" x="0" y="0" z="0">
+      <origin xyz="0 0 0" rpy="0 0 0"/>
+    </xacro:inertial_box>
+</link>
+<joint name="chassis_battery_joint" type="fixed">
+    <parent link="chassis"/>
+    <child link="battery"/>
+    <origin xyz="${-28 * 0.001} 0 ${1.7 * 0.001}"/>
 </joint>
 <!-- Left wheel -->
-<link name="left_motor_mount">
-  <visual>
-    <origin xyz="${10 * 0.001} ${3.375 * 0.001} ${0 * 0.001}" rpy="0 0 0"/>
-    <geometry>
-      <mesh filename="file://$(find cobalt)/description/meshes/motor_mount.stl" scale="0.001 0.001 0.001"/>
-    </geometry>
-    <material name="black"/>
-  </visual>
-</link>
-<joint name="left_motor_mount_joint" type="fixed">
-  <origin xyz="${10 * 0.001} ${32 * 0.001} 0" rpy="0 0 ${pi}"/>
-  <parent link="chassis"/>
-  <child link="left_motor_mount"/>
-</joint>
 <link name="left_wheel">
   <visual>
-    <origin xyz="0 0 ${5 * 0.001}" rpy="${pi/2} 0 0"/>
+    <origin xyz="0 0 0" rpy="0 0 0"/>
     <geometry>
       <mesh filename="file://$(find cobalt)/description/meshes/tire.stl" scale="0.001 0.001 0.001"/>
@@ -56,85 +66,23 @@
   </visual>
   <collision>
-    <origin xyz="0 ${-5 * 0.001} ${5 * 0.001}" rpy="${pi/2} 0 0"/>
+    <origin xyz="0 0 ${5 * 0.001}" rpy="0 0 0"/>
     <geometry>
       <cylinder length="${10 * 0.001}" radius="${21 * 0.001}"/>
     </geometry>
   </collision>
-  <xacro:inertial_cylinder mass="0.2" length="${10  * 0.001}" radius="${21 * 0.001}">
-    <origin xyz="0 ${-5 * 0.001} ${5 * 0.001}" rpy="${pi/2} 0 0"/>
+  <xacro:inertial_cylinder mass="0.008" length="${10  * 0.001}" radius="${21 * 0.001}">
+    <origin xyz="0 0 0" rpy="0 0 0"/>
   </xacro:inertial_cylinder>
 </link>
 <joint name="left_wheel_joint" type="continuous">
-  <origin xyz="${10 * 0.001} ${(-3.125 - 0.5) * 0.001} 0" rpy="0 0 0"/>
-  <parent link="left_motor_mount"/>
+  <origin xyz="0 ${35.4 * 0.001} 0" rpy="${-pi/2} 0 0"/>
+  <parent link="base_link"/>
   <child link="left_wheel"/>
-  <axis xyz="0.0 -1.0 0.0"/>
+  <axis xyz="0.0 0.0 1.0"/>
 </joint>
-<!--
-<link name="left_motor_mount">
-  <visual>
-    <origin xyz="0.01 -0.0318 -0.0129" rpy="0 0 0"/>
-    <geometry>
-      <mesh filename="file://$(find cobalt)/description/meshes/motor_mount.stl" scale="0.001 0.001 0.001"/>
-    </geometry>
-    <material name="black"/>
-  </visual>
-  <collision>
-    <origin xyz="0.01 -0.0318 -0.0129" rpy="0 0 0"/>
-    <geometry>
-      <mesh filename="file://$(find cobalt)/description/meshes/motor_mount.stl" scale="0.001 0.001 0.001"/>
-    </geometry>
-  </collision>
-</link>
-<link name="left_wheel">
-  <inertial>
-    <origin xyz="0 0 0" rpy="0 0 0"/>
-    <mass value="0.09628204164313305"/>
-    <inertia ixx="1.1e-05" iyy="2e-05" izz="1.1e-05" ixy="-0.0" iyz="0.0" ixz="0.0"/>
-  </inertial>
-  <visual>
-    <origin xyz="0.0 0.0 0.0" rpy="0 0 0"/>
-    <geometry>
-      <mesh filename="file://$(find cobalt)/description/meshes/left_wheel.stl" scale="0.001 0.001 0.001"/>
-    </geometry>
-    <material name="yellow"/>
-  </visual>
-  <collision>
-    <origin xyz="0.0 0.0 0.0" rpy="0 0 0"/>
-    <geometry>
-      <mesh filename="file://$(find cobalt)/description/meshes/left_wheel.stl" scale="0.001 0.001 0.001"/>
-    </geometry>
-  </collision>
-</link>
-<joint name="left_motor_mount_joint" type="fixed">
-  <origin xyz="-0.01 0.0318 0.0129" rpy="0 0 0"/>
-  <parent link="chassis"/>
-  <child link="left_motor_mount"/>
-</joint>
-<joint name="left_wheel_joint" type="continuous">
-  <origin xyz="0.01 0.002925 0.01695" rpy="0 0 0"/>
-  <parent link="left_motor_mount"/>
-  <child link="left_wheel"/>
-  <axis xyz="0.0 -1.0 0.0"/>
-</joint>
--->
 <!-- Right wheel -->
-<link name="right_motor_mount">
-  <visual>
-    <origin xyz="${10 * 0.001} ${3.375 * 0.001} ${0 * 0.001}" rpy="0 0 0"/>
-    <geometry>
-      <mesh filename="file://$(find cobalt)/description/meshes/motor_mount.stl" scale="0.001 0.001 0.001"/>
-    </geometry>
-    <material name="black"/>
-  </visual>
-</link>
-<joint name="right_motor_mount_joint" type="fixed">
-  <origin xyz="${-10 * 0.001} ${-32 * 0.001} 0" rpy="0 0 0"/>
-  <parent link="chassis"/>
-  <child link="right_motor_mount"/>
-</joint>
 <link name="right_wheel">
   <visual>
-    <origin xyz="0 0 ${5 * 0.001}" rpy="${pi/2} 0 0"/>
+    <origin xyz="0 0 0" rpy="0 0 0"/>
     <geometry>
       <mesh filename="file://$(find cobalt)/description/meshes/tire.stl" scale="0.001 0.001 0.001"/>
@@ -143,122 +91,18 @@
   </visual>
   <collision>
-    <origin xyz="0 ${-5 * 0.001} ${5 * 0.001}" rpy="${pi/2} 0 0"/>
+    <origin xyz="0 0 ${5 * 0.001}" rpy="0 0 0"/>
     <geometry>
       <cylinder length="${10 * 0.001}" radius="${21 * 0.001}"/>
     </geometry>
   </collision>
-  <xacro:inertial_cylinder mass="0.2" length="${10  * 0.001}" radius="${21 * 0.001}">
-    <origin xyz="0 ${-5 * 0.001} ${5 * 0.001}" rpy="${pi/2} 0 0"/>
+  <xacro:inertial_cylinder mass="0.008" length="${10  * 0.001}" radius="${21 * 0.001}">
+    <origin xyz="0 0 0" rpy="0 0 0"/>
   </xacro:inertial_cylinder>
 </link>
 <joint name="right_wheel_joint" type="continuous">
-  <origin xyz="${10 * 0.001} ${(-3.125 - 0.5) * 0.001} 0" rpy="0 0 0"/>
-  <parent link="right_motor_mount"/>
+  <origin xyz="0 ${-35.4 * 0.001} 0" rpy="${pi/2} 0 0"/>
+  <parent link="base_link"/>
   <child link="right_wheel"/>
-  <axis xyz="0.0 1.0 0.0"/>
+  <axis xyz="0.0 0.0 -1.0"/>
 </joint>
-<!--
-<link name="right_motor_mount">
-  <inertial>
-    <origin xyz="0.009999999999998756 0.005007703274406541 0.0071826271016223586" rpy="0 0 0"/>
-    <mass value="0.013283963856808287"/>
-    <inertia ixx="1e-06" iyy="1e-06" izz="1e-06" ixy="-0.0" iyz="-0.0" ixz="-0.0"/>
-  </inertial>
-  <visual>
-    <origin xyz="0.01 0.0322 -0.0129" rpy="0 0 0"/>
-    <geometry>
-      <mesh filename="file://$(find cobalt)/description/meshes/right_motor_mount.stl" scale="0.001 0.001 0.001"/>
-    </geometry>
-    <material name="black"/>
-  </visual>
-  <collision>
-    <origin xyz="0.01 0.0322 -0.0129" rpy="0 0 0"/>
-    <geometry>
-      <mesh filename="file://$(find cobalt)/description/meshes/right_motor_mount.stl" scale="0.001 0.001 0.001"/>
-    </geometry>
-  </collision>
-</link>
-<link name="right_wheel">
-  <inertial>
-    <origin xyz="1.155986334056513e-13 -0.07594400200685048 -0.011699240852793388" rpy="0 0 0"/>
-    <mass value="0.09628204164313274"/>
-    <inertia ixx="1.1e-05" iyy="2e-05" izz="1.1e-05" ixy="0.0" iyz="0.0" ixz="-0.0"/>
-  </inertial>
-  <visual>
-    <origin xyz="0.0 -0.035125 -0.02985" rpy="0 0 0"/>
-    <geometry>
-      <mesh filename="file://$(find cobalt)/description/meshes/right_wheel.stl" scale="0.001 0.001 0.001"/>
-    </geometry>
-    <material name="yellow"/>
-  </visual>
-  <collision>
-    <origin xyz="0.0 -0.035125 -0.02985" rpy="0 0 0"/>
-    <geometry>
-      <mesh filename="file://$(find cobalt)/description/meshes/right_wheel.stl" scale="0.001 0.001 0.001"/>
-    </geometry>
-  </collision>
-</link>
-<joint name="right_motor_mount_joint" type="fixed">
-  <origin xyz="-0.01 -0.0322 0.0129" rpy="0 0 0"/>
-  <parent link="chassis"/>
-  <child link="right_motor_mount"/>
-</joint>
-<joint name="right_wheel_joint" type="continuous">
-  <origin xyz="0.01 0.067325 0.01695" rpy="0 0 0"/>
-  <parent link="right_motor_mount"/>
-  <child link="right_wheel"/>
-  <axis xyz="-0.0 1.0 -0.0"/>
-</joint>
--->
-<!-- Caster wheel -->
-<link name="caster_wheel">
-  <visual>
-    <origin xyz="${42 * 0.001} ${12 * 0.001} ${-11.7 * 0.001}" rpy="0 0 0"/>
-    <geometry>
-      <mesh filename="file://$(find cobalt)/description/meshes/caster_wheel.stl" scale="0.001 0.001 0.001"/>
-    </geometry>
-    <material name="black"/>
-  </visual>
-  <collision>
-    <origin xyz="${42 * 0.001} ${12 * 0.001} ${-11.7 * 0.001}" rpy="0 0 0"/>
-    <geometry>
-      <mesh filename="file://$(find cobalt)/description/meshes/caster_wheel.stl" scale="0.001 0.001 0.001"/>
-    </geometry>
-  </collision>
-  <xacro:inertial_cylinder mass="0.2" length="${10  * 0.001}" radius="${21 * 0.001}">
-    <origin xyz="${42 * 0.001} ${12 * 0.001} ${-11.7 * 0.001}" rpy="0 0 0"/>
-  </xacro:inertial_cylinder>
-</link>
-<joint name="caster_wheel_joint" type="fixed">
-  <origin xyz="${-42 * 0.001} ${-12 * 0.001} 0" rpy="0 0 0"/>
-  <parent link="chassis"/>
-  <child link="caster_wheel"/>
-</joint>
-<!--
-<link name="caster_wheel">
-  <inertial>
-    <origin xyz="-3.2959746043559335e-15 0.01200000000012692 -0.005472929175792768" rpy="0 0 0"/>
-    <mass value="0.01927290082472035"/>
-    <inertia ixx="1e-06" iyy="0.0" izz="1e-06" ixy="-0.0" iyz="0.0" ixz="0.0"/>
-  </inertial>
-  <visual>
-    <origin xyz="0.042 0.0122 -0.0117" rpy="0 0 0"/>
-    <geometry>
-      <mesh filename="file://$(find cobalt)/description/meshes/caster_wheel.stl" scale="0.001 0.001 0.001"/>
-    </geometry>
-    <material name="black"/>
-  </visual>
-  <collision>
-    <origin xyz="0.042 0.0122 -0.0117" rpy="0 0 0"/>
-    <geometry>
-      <mesh filename="file://$(find cobalt)/description/meshes/caster_wheel.stl" scale="0.001 0.001 0.001"/>
-    </geometry>
-  </collision>
-</link>
-<joint name="caster_wheel_joint" type="fixed">
-  <origin xyz="-0.042 -0.0122 0.0117" rpy="0 0 0"/>
-  <parent link="chassis"/>
-  <child link="caster_wheel"/>
-</joint>
--->
 </robot>

Commit message: Package rename

File: description/urdf/urdf.xacro (robot description, xacro)
@@ -1,9 +1,8 @@
 <?xml version="1.0" ?>
 <robot name="urdf" xmlns:xacro="http://www.ros.org/wiki/xacro">
-<xacro:include filename="$(find cobalt)/description/urdf/inertia.xacro" />
-<xacro:include filename="$(find cobalt)/description/urdf/materials.xacro" />
-<xacro:include filename="$(find cobalt)/description/urdf/urdf.trans" />
-<xacro:include filename="$(find cobalt)/description/urdf/urdf.gazebo" />
-<xacro:include filename="$(find cobalt)/description/urdf/control.xacro" />
+<xacro:include filename="$(find cobalt_simulation)/description/urdf/inertia.xacro" />
+<xacro:include filename="$(find cobalt_simulation)/description/urdf/materials.xacro" />
+<xacro:include filename="$(find cobalt_simulation)/description/urdf/urdf.gazebo" />
+<xacro:include filename="$(find cobalt_simulation)/description/urdf/control.xacro" />
 <!-- Base link -->
 <link name="base_link">
@@ -14,5 +13,5 @@
         <origin xyz="0 0 ${1.7 * 0.001}" rpy="${pi} 0 0"/>
         <geometry>
-          <mesh filename="file://$(find cobalt)/description/meshes/base_link.stl" scale="0.001 0.001 0.001"/>
+          <mesh filename="file://$(find cobalt_simulation)/description/meshes/base_link.stl" scale="0.001 0.001 0.001"/>
         </geometry>
         <material name="black"/>
@@ -37,5 +36,5 @@
         <origin xyz="0 0 0" rpy="0 0 0"/>
         <geometry>
-            <mesh filename="file://$(find cobalt)/description/meshes/battery.stl" scale="0.001 0.001 0.001"/>
+            <mesh filename="file://$(find cobalt_simulation)/description/meshes/battery.stl" scale="0.001 0.001 0.001"/>
         </geometry>
         <material name="black"/>
@@ -61,5 +60,5 @@
     <origin xyz="0 0 0" rpy="0 0 0"/>
     <geometry>
-      <mesh filename="file://$(find cobalt)/description/meshes/tire.stl" scale="0.001 0.001 0.001"/>
+      <mesh filename="file://$(find cobalt_simulation)/description/meshes/tire.stl" scale="0.001 0.001 0.001"/>
     </geometry>
     <material name="yellow"/>
@@ -86,5 +85,5 @@
     <origin xyz="0 0 0" rpy="0 0 0"/>
     <geometry>
-      <mesh filename="file://$(find cobalt)/description/meshes/tire.stl" scale="0.001 0.001 0.001"/>
+      <mesh filename="file://$(find cobalt_simulation)/description/meshes/tire.stl" scale="0.001 0.001 0.001"/>
     </geometry>
     <material name="yellow"/>
